Commit message: adding rw files and config type

File: src/robot_properties_bolt/resources/xacro/bolt_rw.urdf.xacro (robot description, xacro)
@@ -14,5 +14,5 @@
   <xacro:include filename="bolt_rw.xacro"/>
   <!-- Include the fully parametrized bolt -->
-  <xacro:bolt_full
+  <xacro:bolt_rw_full
       mesh_ext="${mesh_ext}"
       color_name="${color_name}"

File: src/robot_properties_bolt/resources/xacro/bolt_rw.xacro (robot description, xacro)
@@ -5,5 +5,5 @@
   xmlns:sensor="http://playerstage.sourceforge.net/gazebo/xmlschema/#sensor"
   xmlns:xacro="http://playerstage.sourceforge.net/gazebo/xmlschema/#interface">
-  <xacro:macro name="bolt_full" params="mesh_ext color_name color opacity new_leg has_passive_ankle">
+  <xacro:macro name="bolt_rw_full" params="mesh_ext color_name color opacity new_leg has_passive_ankle">
     <!-- This file is based on: https://atlas.is.localnet/confluence/display/AMDW/Quadruped+URDF+Files -->
     <link name="base_link">
@@ -44,4 +44,12 @@
       </contact>
     </link> <!-- END BASE LINK -->
+    <!-- Include the reaction wheel -->
+    <xacro:include filename="rw_4004.xacro"/>
+    <!-- Include the upper body -->
+    <xacro:rw_4004
+        mesh_ext="${mesh_ext}"
+        color_name="${color_name}"
+        color="${color}"
+        opacity="${opacity}"/>
     <!-- Include the legs -->
     <xacro:include filename="leg.xacro"/>
